File: mu80-dit.kicad_sch (KiCad schematic)
At the start: 21 parts, among them J1 Conn_01x06_Male, J2 Conn_01x02_Male, U1 TOTX-177L, U2 74FST3257DTR2G, U4 74HCT7731, U5 74HCT74D

Commit message: update flipflop part
Parts:
- U5: value 74HCT74D -> SN74HCT74
Changed lines of the file:
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@@
     (in_bom yes) (on_board yes) (fields_autoplaced)
     (property "Reference" "U5" (id 0) (at 105.41 45.72 0))
-    (property "Value" "74HCT74D" (id 1) (at 105.41 48.26 0))
+    (property "Value" "SN74HCT74" (id 1) (at 105.41 48.26 0))
     (property "Footprint" "Package_SO:SO-14_3.9x8.65mm_P1.27mm" (id 2) (at 133.51 100.92 0)
       (effects (font (size 1.27 1.27)) (justify left bottom) hide)
@@
     )
     (path "/e9ecf0cb-ce8c-4426-a520-b03e079cae72"
-      (reference "U5") (unit 1) (value "74HCT74D") (footprint "Package_SO:SO-14_3.9x8.65mm_P1.27mm")
+      (reference "U5") (unit 1) (value "SN74HCT74") (footprint "Package_SO:SO-14_3.9x8.65mm_P1.27mm")
     )
     (path "/cbb89bd7-29b1-418d-bb17-a5e078b16f28"
